File: Sofle_v3/PCB/SofleKeyboard.kicad_pcb (KiCad board)
At the start: 2 copper layers, 141.4 x 114.1 mm, 99 parts, among them J1 LED, J2 4PIN, J3 OLED, J4 key leds, J5 backlight sel, J6 indicator bypass, P1 i2c_pin, P2 i2c_pin, SW1 SW_PUSH-MX_W_LED, SW10 SW_PUSH-MX_W_LED, SW11 SW_PUSH-MX_W_LED, SW12 SW_PUSH-MX_W_LED, SW13 SW_PUSH-MX_W_LED, SW14 SW_PUSH-MX_W_LED, SW15 SW_PUSH-MX_W_LED, SW16 SW_PUSH-MX_W_LED, SW17 SW_PUSH-MX_W_LED, SW18 SW_PUSH-MX_W_LED, SW19 SW_PUSH-MX_W_LED, SW2 SW_PUSH-MX_W_LED, SW20 SW_PUSH-MX_W_LED, SW21 SW_PUSH-MX_W_LED, SW22 SW_PUSH-MX_W_LED, SW23 SW_PUSH-MX_W_LED, SW24 SW_PUSH-MX_W_LED, SW25 Rotary_Encoder_Switch, SW26 SW_PUSH-MX_W_LED, SW27 SW_PUSH-MX_W_LED, SW28 SW_PUSH-MX_W_LED, SW29 SW_PUSH-MX_W_LED, SW3 SW_PUSH-MX_W_LED, SW30 SW_PUSH-MX_W_LED, SW4 SW_PUSH-MX_W_LED, SW5 SW_PUSH-MX_W_LED, SW6 SW_PUSH-MX_W_LED, SW7 SW_PUSH-MX_W_LED, SW8 SW_PUSH-MX_W_LED, SW9 SW_PUSH-MX_W_LED, U1 ProMicro

Commit message: design: routing and schematic beatifications
Parts:
- D31, D32, D33, D34, D35, D36, D37: footprint LED_SMD:SK6812MINI_underglow_dev -> SofleRGB:LED_WS2812B_TwoSided
- J2: footprint SofleKeyboard-footprint:MJ-4PP-9 -> SofleRGB:WM2211210044
- RSW1: footprint SofleKeyboard-footprint:TACT_SWITCH_TVBP06 -> SofleRGB:TPS635-1B43D
- moved D30 43.7 mm to (169.5, 120.5), turned to -90 degrees
- moved D29 23.3 mm to (149.0, 124.0), turned to -90 degrees
- moved D19 17.0 mm to (129.0, 103.0)
- moved D33 14.0 mm to (185.5, 60.0), turned to -90 degrees
- moved J5 9.89 mm to (166.5, 113.5), turned to 180 degrees
- moved D31 7.57 mm to (113.0, 60.5), turned to -90 degrees
- moved D32 7.50 mm to (151.0, 53.8), turned to 90 degrees
- moved D27 5.14 mm to (114.5, 117.5), turned to -164 degrees
- moved D28 4.55 mm to (130.0, 122.5), turned to -90 degrees
- moved J2 3.95 mm to (88.0, 89.6), turned to 0 degrees
- moved D26 3.65 mm to (97.2, 124.2), turned to -150 degrees
- moved D24 3.30 mm to (206.5, 114.0)
- moved D11 3.23 mm to (188.0, 76.0)
- moved D34 3.17 mm to (107.5, 127.0), turned to 106 degrees
- moved D18 2.83 mm to (207.0, 95.0)
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Connections:
- net Net-(D1-Pad2) renamed /SW1_D
- net Net-(D10-Pad2) renamed /SW10_D
- net Net-(D11-Pad2) renamed /SW11_D
- net Net-(D12-Pad2) renamed /SW12_D
- net Net-(D13-Pad2) renamed /SW13_D
- net Net-(D14-Pad2) renamed /SW14_D
- net Net-(D15-Pad2) renamed /SW15_D
- net Net-(D16-Pad2) renamed /SW16_D
- net Net-(D17-Pad2) renamed /SW17_D
- net Net-(D18-Pad2) renamed /SW18_D
- net Net-(D19-Pad2) renamed /SW19_D
- net Net-(D2-Pad2) renamed /SW2_D
- net Net-(D20-Pad2) renamed /SW20_D
- net Net-(D21-Pad2) renamed /SW21_D
- net Net-(D22-Pad2) renamed /SW22_D
- net Net-(D23-Pad2) renamed /SW23_D
- net Net-(D24-Pad2) renamed /SW24_D
- net Net-(D26-Pad2) renamed /SW26_D
- net Net-(D27-Pad2) renamed /SW27_D
- net Net-(D28-Pad2) renamed /SW28_D
- net Net-(D29-Pad2) renamed /SW29_D
- net Net-(D3-Pad2) renamed /SW3_D
- net Net-(D30-Pad2) renamed /SW30_D
- net Net-(D4-Pad2) renamed /SW4_D
- net Net-(D5-Pad2) renamed /SW5_D
- net Net-(D6-Pad2) renamed /SW6_D
- net Net-(D7-Pad2) renamed /SW7_D
- net Net-(D8-Pad2) renamed /SW8_D
- net Net-(D9-Pad2) renamed /SW9_D
- net SW25A renamed col5
- net SW25B renamed /SW25B
- D31 pad 1: Net-(D31-Pad1) -> VCC
- D31 pad 2: GND -> Net-(D31-Pad2)
- D31 pad 3: Net-(D31-Pad3) -> GND
- D31 pad 4: VCC -> Net-(D31-Pad4)
- D32 pad 1: Net-(D31-Pad3) -> VCC
- D32 pad 2: GND -> Net-(D31-Pad4)
- D32 pad 3: Net-(D32-Pad3) -> GND
- D32 pad 4: VCC -> Net-(D32-Pad4)
- D33 pad 1: Net-(D32-Pad3) -> VCC
- D33 pad 2: GND -> Net-(D32-Pad4)
- D33 pad 3: /underglow -> GND
- D33 pad 4: VCC -> /underglow
- D34 pad 1: Net-(D34-Pad1) -> VCC
- D34 pad 2: GND -> Net-(D34-Pad2)
- D34 pad 3: Net-(D31-Pad1) -> GND
- D34 pad 4: VCC -> Net-(D31-Pad2)
- D35 pad 1: Net-(D35-Pad1) -> VCC
- D35 pad 2: GND -> Net-(D35-Pad2)
- D35 pad 3: Net-(D34-Pad1) -> GND
- D35 pad 4: VCC -> Net-(D34-Pad2)
- D36 pad 1: Net-(D36-Pad1) -> VCC
- D36 pad 2: GND -> Net-(D36-Pad2)
- D36 pad 3: Net-(D35-Pad1) -> GND
- D36 pad 4: VCC -> Net-(D35-Pad2)
- D37 pad 2: GND -> VCC
- D37 pad 4: VCC -> GND
- J5 pad 2: Net-(D36-Pad1) -> Net-(D36-Pad2)
- SW1 pad 1: Net-(SW1-Pad1) -> VCC
- SW1 pad 2: GND -> Net-(SW1-Pad2)
- SW1 pad 3: Net-(SW1-Pad3) -> GND
- SW1 pad 4: VCC -> Net-(SW1-Pad4)
- SW10 pad 1: Net-(SW10-Pad1) -> VCC
- SW10 pad 2: GND -> Net-(SW10-Pad2)
- SW10 pad 3: Net-(SW10-Pad3) -> GND
- SW10 pad 4: VCC -> Net-(SW10-Pad4)
- SW11 pad 1: Net-(SW11-Pad1) -> VCC
- SW11 pad 2: GND -> Net-(SW11-Pad2)
- SW11 pad 3: Net-(SW11-Pad3) -> GND
- SW11 pad 4: VCC -> Net-(SW11-Pad4)
- SW12 pad 1: Net-(SW12-Pad1) -> VCC
- SW12 pad 2: GND -> Net-(SW12-Pad2)
- SW12 pad 3: Net-(SW12-Pad3) -> GND
- SW12 pad 4: VCC -> Net-(SW12-Pad4)
- SW13 pad 1: Net-(SW13-Pad1) -> VCC
- SW13 pad 2: GND -> Net-(SW13-Pad2)
- SW13 pad 3: Net-(SW13-Pad3) -> GND
- SW13 pad 4: VCC -> Net-(SW13-Pad4)
- SW14 pad 1: Net-(SW14-Pad1) -> VCC
- SW14 pad 2: GND -> Net-(SW14-Pad2)
- SW14 pad 3: Net-(SW14-Pad3) -> GND
- SW14 pad 4: VCC -> Net-(SW14-Pad4)
- SW15 pad 1: Net-(SW15-Pad1) -> VCC
- SW15 pad 2: GND -> Net-(SW15-Pad2)
- SW15 pad 3: Net-(SW15-Pad3) -> GND
- SW15 pad 4: VCC -> Net-(SW15-Pad4)
- SW16 pad 1: Net-(SW10-Pad3) -> VCC
- SW16 pad 2: GND -> Net-(SW16-Pad2)
- SW16 pad 3: Net-(SW16-Pad3) -> GND
- SW16 pad 4: VCC -> Net-(SW10-Pad2)
- SW17 pad 1: Net-(SW17-Pad1) -> VCC
- SW17 pad 2: GND -> Net-(SW11-Pad4)
- SW17 pad 3: Net-(SW11-Pad1) -> GND
- SW17 pad 4: VCC -> Net-(SW17-Pad4)
- SW18 pad 1: Net-(SW12-Pad3) -> VCC
- SW18 pad 2: GND -> Net-(SW18-Pad2)
- SW18 pad 3: Net-(SW18-Pad3) -> GND
- SW18 pad 4: VCC -> Net-(SW12-Pad2)
- SW19 pad 1: unconnected-(SW19-Pad1) -> VCC
- SW19 pad 2: GND -> Net-(SW13-Pad4)
- SW19 pad 3: Net-(SW13-Pad1) -> GND
- SW19 pad 4: VCC -> unconnected-(SW19-Pad4)
- SW2 pad 1: Net-(SW1-Pad3) -> VCC
- SW2 pad 2: GND -> Net-(SW2-Pad2)
- SW2 pad 3: Net-(SW2-Pad3) -> GND
- SW2 pad 4: VCC -> Net-(SW1-Pad2)
- SW20 pad 1: Net-(SW14-Pad3) -> VCC
- SW20 pad 2: GND -> Net-(SW20-Pad2)
- SW20 pad 3: Net-(SW20-Pad3) -> GND
- SW20 pad 4: VCC -> Net-(SW14-Pad2)
- SW21 pad 1: Net-(SW21-Pad1) -> VCC
- SW21 pad 2: GND -> Net-(SW15-Pad4)
- SW21 pad 3: Net-(SW15-Pad1) -> GND
- SW21 pad 4: VCC -> Net-(SW21-Pad4)
- SW22 pad 1: Net-(SW16-Pad3) -> VCC
- SW22 pad 2: GND -> Net-(SW22-Pad2)
- SW22 pad 3: Net-(SW22-Pad3) -> GND
- SW22 pad 4: VCC -> Net-(SW16-Pad2)
- SW23 pad 1: Net-(SW23-Pad1) -> VCC
- SW23 pad 2: GND -> Net-(SW17-Pad4)
- SW23 pad 3: Net-(SW17-Pad1) -> GND
- SW23 pad 4: VCC -> Net-(SW23-Pad4)
- SW24 pad 1: Net-(SW18-Pad3) -> VCC
- SW24 pad 2: GND -> Net-(SW24-Pad2)
- SW24 pad 3: Net-(SW24-Pad3) -> GND
- SW24 pad 4: VCC -> Net-(SW18-Pad2)
- SW26 pad 1: Net-(SW20-Pad3) -> VCC
- SW26 pad 2: GND -> Net-(SW26-Pad2)
- SW26 pad 3: Net-(SW26-Pad3) -> GND
- SW26 pad 4: VCC -> Net-(SW20-Pad2)
- SW27 pad 1: Net-(SW26-Pad3) -> VCC
- SW27 pad 2: GND -> Net-(SW21-Pad4)
- SW27 pad 3: Net-(SW21-Pad1) -> GND
- SW27 pad 4: VCC -> Net-(SW26-Pad2)
- SW28 pad 1: Net-(SW22-Pad3) -> VCC
- SW28 pad 2: GND -> Net-(SW28-Pad2)
- SW28 pad 3: Net-(SW28-Pad3) -> GND
- SW28 pad 4: VCC -> Net-(SW22-Pad2)
- SW29 pad 1: Net-(SW28-Pad3) -> VCC
- SW29 pad 2: GND -> Net-(SW23-Pad4)
- SW29 pad 3: Net-(SW23-Pad1) -> GND
- SW29 pad 4: VCC -> Net-(SW28-Pad2)
- SW3 pad 1: Net-(SW3-Pad1) -> VCC
- SW3 pad 2: GND -> Net-(SW3-Pad2)
- SW3 pad 3: Net-(SW3-Pad3) -> GND
- SW3 pad 4: VCC -> Net-(SW3-Pad4)
- SW30 pad 1: Net-(SW24-Pad3) -> VCC
- SW30 pad 2: GND -> /backlight
- SW30 pad 3: /backlight -> GND
- SW30 pad 4: VCC -> Net-(SW24-Pad2)
- SW4 pad 1: Net-(SW3-Pad3) -> VCC
- SW4 pad 2: GND -> Net-(SW10-Pad4)
- SW4 pad 3: Net-(SW10-Pad1) -> GND
- SW4 pad 4: VCC -> Net-(SW3-Pad2)
- SW5 pad 1: Net-(SW11-Pad3) -> VCC
- SW5 pad 2: GND -> Net-(SW5-Pad2)
- SW5 pad 3: Net-(SW5-Pad3) -> GND
- SW5 pad 4: VCC -> Net-(SW11-Pad2)
- SW6 pad 1: Net-(SW5-Pad3) -> VCC
- SW6 pad 2: GND -> Net-(SW12-Pad4)
- SW6 pad 3: Net-(SW12-Pad1) -> GND
- SW6 pad 4: VCC -> Net-(SW5-Pad2)
- SW7 pad 1: Net-(SW13-Pad3) -> VCC
- SW7 pad 2: GND -> Net-(SW1-Pad4)
- SW7 pad 3: Net-(SW1-Pad1) -> GND
- SW7 pad 4: VCC -> Net-(SW13-Pad2)
- SW8 pad 1: Net-(SW2-Pad3) -> VCC
- SW8 pad 2: GND -> Net-(SW14-Pad4)
- SW8 pad 3: Net-(SW14-Pad1) -> GND
- SW8 pad 4: VCC -> Net-(SW2-Pad2)
- SW9 pad 1: Net-(SW15-Pad3) -> VCC
- SW9 pad 2: GND -> Net-(SW3-Pad4)
- SW9 pad 3: Net-(SW3-Pad1) -> GND
- SW9 pad 4: VCC -> Net-(SW15-Pad2)
Routing:
- net VCC: track 0.00 -> 925.3 mm, vias 0 -> 51
- net col3: track 0.00 -> 244.2 mm, vias 0 -> 6
- net col4: track 0.00 -> 224.0 mm, vias 0 -> 6
- net col2: track 0.00 -> 188.8 mm, vias 0 -> 5
- net col0: track 0.00 -> 179.2 mm, vias 0 -> 5
- net col1: track 0.00 -> 178.3 mm, vias 0 -> 6
- net row4: track 0.00 -> 157.5 mm, vias 0 -> 6
- net col5: track 0.00 -> 143.2 mm, vias 0 -> 6
- net row1: track 0.00 -> 112.9 mm, vias 0 -> 5
- net row0: track 0.00 -> 112.5 mm, vias 0 -> 6
- net row3: track 0.00 -> 112.0 mm, vias 0 -> 6
- net row2: track 0.00 -> 111.2 mm, vias 0 -> 5
- net LED: track 0.00 -> 61.3 mm, vias 0 -> 2
- net SDA: track 0.00 -> 54.9 mm, vias 0 -> 3
- net GND: track 0.00 -> 54.7 mm, vias 0 -> 2
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Other:
- board text added: "Yet another variant by Jesko Edzards and Jan Schoneberg Based on Sofle RGB by Dane Evans, original by Josef Adamacik"
- board text removed: "Sofle RGB by Dane Evans, original by Josef Adamacik"
- board text removed: "Sofle RGB v2.1, Dane Evans"
