File: Sofle_v3/PCB/SofleKeyboard.kicad_sch (KiCad schematic)
At the start: 145 parts, among them J1 LED, J2 4PIN, J3 OLED, J4 key leds, J5 backlight sel, J6 indicator bypass, P1 i2c_pin, P2 i2c_pin, SW1 SW_PUSH-MX_W_LED, SW10 SW_PUSH-MX_W_LED, SW11 SW_PUSH-MX_W_LED, SW12 SW_PUSH-MX_W_LED, SW13 SW_PUSH-MX_W_LED, SW14 SW_PUSH-MX_W_LED, SW15 SW_PUSH-MX_W_LED, SW16 SW_PUSH-MX_W_LED, SW17 SW_PUSH-MX_W_LED, SW18 SW_PUSH-MX_W_LED, SW19 SW_PUSH-MX_W_LED, SW2 SW_PUSH-MX_W_LED, SW20 SW_PUSH-MX_W_LED, SW21 SW_PUSH-MX_W_LED, SW22 SW_PUSH-MX_W_LED, SW23 SW_PUSH-MX_W_LED, SW24 SW_PUSH-MX_W_LED, SW25 Rotary_Encoder_Switch, SW26 SW_PUSH-MX_W_LED, SW27 SW_PUSH-MX_W_LED, SW28 SW_PUSH-MX_W_LED, SW29 SW_PUSH-MX_W_LED, SW3 SW_PUSH-MX_W_LED, SW30 SW_PUSH-MX_W_LED, SW4 SW_PUSH-MX_W_LED, SW5 SW_PUSH-MX_W_LED, SW6 SW_PUSH-MX_W_LED, SW7 SW_PUSH-MX_W_LED, SW8 SW_PUSH-MX_W_LED, SW9 SW_PUSH-MX_W_LED, U100 ProMicroDualSided

Commit message: production files added
Other:
- note removed: "TODO: - Check unglow led position - Encoder daughterboard - DRC - Check encoder side matrix Erledigt: - Headphone Jack footprint - Mahority of routing - Reset button footprint - Underglow LED positioning (carefull with mounting holes - enough space to them)"
Changed lines of the file:
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@@
     (stroke (width 0) (type default) (color 0 0 0 0))
-  )
-  (text "TODO:\n- Check unglow led position\n- Encoder daughterboard\n- DRC\n- Check encoder side matrix\n\nErledigt:\n- Headphone Jack footprint\n- Mahority of routing\n- Reset button footprint\n- Underglow LED positioning (carefull with mounting holes - enough space to them)"
-    (at 22.86 254 0)
-    (effects (font (size 1.27 1.27)) (justify left bottom))
   )
   (label "SW25A" (at 63.5 214.63 180)
