File: Sofle_v3/DaughterBoard/DaughterBoard.kicad_pcb (KiCad board)
At the start: 2 copper layers, 25.5 x 18 mm, 2 parts, among them SW1 RotaryEncoder_Switch, SW2 RotaryEncoder_Switch

Commit message: design: daughter board update
Parts:
- moved SW1 1.03 mm to (147.4, 80.5)
Routing:
- net Net-(SW1-PadS2): track 6.07 -> 41.1 mm
- net Net-(SW1-PadB): track 5.63 -> 35.9 mm
- net Net-(SW1-PadC): track 6.99 -> 33.2 mm
- net Net-(SW1-PadD): track 4.45 -> 29.4 mm
- net Net-(SW1-PadA): track 8.04 -> 32.7 mm
- net Net-(SW1-PadS1): track 9.45 -> 30.9 mm
Other:
- board size 25.5 x 18 mm -> 26.2 x 19.5 mm

Commit message: production files added
Changed lines of the file:
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@@
       (net 5 "Net-(SW1-PadS2)") (pinfunction "S2") (pintype "passive"))
   )
+  (gr_poly
+    (pts
+      (xy 149.714372 91.808)
+      (xy 134.589372 91.808)
+      (xy 134.589372 72.308)
+      (xy 145.714372 72.308)
+    ) (layer "B.SilkS") (width 0.01) (fill solid))
+  (gr_poly
+    (pts
+      (xy 149.713 91.808)
+      (xy 134.588 91.808)
+      (xy 134.588 72.308)
+      (xy 145.713 72.308)
+    ) (layer "F.SilkS") (width 0.01) (fill solid))
   (segment (start 136.590001 80.790001) (end 140.640002 76.74) (width 0.25) (layer "F.Cu") (net 1))
   (segment (start 140.640002 76.74) (end 141.755 76.74) (width 0.25) (layer "F.Cu") (net 1))
@@
   (segment (start 139.169999 75.710001) (end 140.53 74.35) (width 0.25) (layer "F.Cu") (net 4))
   (segment (start 136.590001 75.710001) (end 139.169999 75.710001) (width 0.25) (layer "F.Cu") (net 4))
+  (segment (start 141.495 78.155) (end 142.220991 78.155) (width 0.25) (layer "B.Cu") (net 4))
+  (segment (start 142.220991 78.155) (end 153.153991 89.088) (width 0.25) (layer "B.Cu") (net 4))
   (segment (start 140.53 77.19) (end 141.495 78.155) (width 0.25) (layer "B.Cu") (net 4))
+  (segment (start 158.162002 89.088) (end 158.840001 88.410001) (width 0.25) (layer "B.Cu") (net 4))
+  (segment (start 153.153991 89.088) (end 158.162002 89.088) (width 0.25) (layer "B.Cu") (net 4))
   (segment (start 140.53 74.35) (end 140.53 77.19) (width 0.25) (layer "B.Cu") (net 4))
-  (segment (start 150.928 86.988) (end 153.028 89.088) (width 0.25) (layer "B.Cu") (net 4))
-  (segment (start 142.220991 78.155) (end 150.928 86.862009) (width 0.25) (layer "B.Cu") (net 4))
-  (segment (start 141.495 78.155) (end 142.220991 78.155) (width 0.25) (layer "B.Cu") (net 4))
-  (segment (start 153.028 89.088) (end 158.162002 89.088) (width 0.25) (layer "B.Cu") (net 4))
-  (segment (start 158.162002 89.088) (end 158.840001 88.410001) (width 0.25) (layer "B.Cu") (net 4))
-  (segment (start 150.928 86.862009) (end 150.928 86.988) (width 0.25) (layer "B.Cu") (net 4))
-  (segment (start 159.028 89.988) (end 160.028 88.988) (width 0.25) (layer "B.Cu") (net 5))
+  (segment (start 152.853 89.988) (end 159.028 89.988) (width 0.25) (layer "B.Cu") (net 5))
   (segment (start 160.028 86.188) (end 159.710001 85.870001) (width 0.25) (layer "B.Cu") (net 5))
+  (segment (start 160.028 88.988) (end 160.028 86.188) (width 0.25) (layer "B.Cu") (net 5))
+  (segment (start 139.128 78.243991) (end 141.579009 80.695) (width 0.25) (layer "B.Cu") (net 5))
   (segment (start 139.991 73.225) (end 139.128 74.088) (width 0.25) (layer "B.Cu") (net 5))
   (segment (start 139.12199 78.250001) (end 139.128 78.243991) (width 0.25) (layer "B.Cu") (net 5))
+  (segment (start 139.128 74.088) (end 139.128 78.243991) (width 0.25) (layer "B.Cu") (net 5))
+  (segment (start 143.56 80.695) (end 152.853 89.988) (width 0.25) (layer "B.Cu") (net 5))
+  (segment (start 159.028 89.988) (end 160.028 88.988) (width 0.25) (layer "B.Cu") (net 5))
+  (segment (start 136.590001 78.250001) (end 139.12199 78.250001) (width 0.25) (layer "B.Cu") (net 5))
+  (segment (start 141.255 73.225) (end 139.991 73.225) (width 0.25) (layer "B.Cu") (net 5))
+  (segment (start 141.579009 80.695) (end 143.56 80.695) (width 0.25) (layer "B.Cu") (net 5))
   (segment (start 159.710001 85.870001) (end 158.840001 85.870001) (width 0.25) (layer "B.Cu") (net 5))
-  (segment (start 151.128 88.688) (end 151.128 88.788) (width 0.25) (layer "B.Cu") (net 5))
-  (segment (start 151.128 88.788) (end 152.328 89.988) (width 0.25) (layer "B.Cu") (net 5))
-  (segment (start 139.128 74.088) (end 139.128 78.243991) (width 0.25) (layer "B.Cu") (net 5))
-  (segment (start 160.028 88.988) (end 160.028 86.188) (width 0.25) (layer "B.Cu") (net 5))
-  (segment (start 141.579009 80.695) (end 143.135 80.695) (width 0.25) (layer "B.Cu") (net 5))
-  (segment (start 136.590001 78.250001) (end 139.12199 78.250001) (width 0.25) (layer "B.Cu") (net 5))
-  (segment (start 143.135 80.695) (end 151.128 88.688) (width 0.25) (layer "B.Cu") (net 5))
-  (segment (start 141.255 73.225) (end 139.991 73.225) (width 0.25) (layer "B.Cu") (net 5))
   (segment (start 142.38 74.35) (end 141.255 73.225) (width 0.25) (layer "B.Cu") (net 5))
-  (segment (start 152.328 89.988) (end 159.028 89.988) (width 0.25) (layer "B.Cu") (net 5))
-  (segment (start 139.128 78.243991) (end 141.579009 80.695) (width 0.25) (layer "B.Cu") (net 5))
   (segment (start 141.755 84.36) (end 152.290864 73.824136) (width 0.25) (layer "F.Cu") (net 6))
   (segment (start 136.590001 88.410001) (end 140.640002 84.36) (width 0.25) (layer "F.Cu") (net 6))
